File: RP2040-PinTest.kicad_pcb (KiCad board)
At the start: 2 copper layers, 57.2 x 53.3 mm, 62 parts, among them J1 Conn_01x02_Socket

Commit message: Moved stuff around.
Routing:
- net GND: track 0.00 -> 27.2 mm, vias 95 -> 97
- net A6: track 36.6 -> 37.3 mm
Changed lines of the file:
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@@
     (effects (font (size 1 1) (thickness 0.15)) (justify top))
   )
+  (segment (start 153.67 105.41) (end 152.4 104.14) (width 0.2) (layer "F.Cu") (net 1))
+  (segment (start 153.67 108.585) (end 153.67 105.41) (width 0.2) (layer "F.Cu") (net 1))
   (via (at 147.955 108.585) (size 0.7) (drill 0.35) (layers "F.Cu" "B.Cu") (free) (net 1))
   (via (at 178.435 109.22) (size 0.7) (drill 0.35) (layers "F.Cu" "B.Cu") (free) (net 1))
@@
   (via (at 173.355 81.28) (size 0.7) (drill 0.35) (layers "F.Cu" "B.Cu") (free) (net 1))
   (via (at 170.18 80.645) (size 0.7) (drill 0.35) (layers "F.Cu" "B.Cu") (free) (net 1))
+  (via (at 152.4 104.14) (size 0.8) (drill 0.4) (layers "F.Cu" "B.Cu") (net 1))
   (via (at 158.115 86.995) (size 0.7) (drill 0.35) (layers "F.Cu" "B.Cu") (free) (net 1))
   (via (at 133.35 86.995) (size 0.7) (drill 0.35) (layers "F.Cu" "B.Cu") (free) (net 1))
+  (via (at 143.51 103.505) (size 0.8) (drill 0.4) (layers "F.Cu" "B.Cu") (net 1))
   (via (at 161.29 118.745) (size 0.7) (drill 0.35) (layers "F.Cu" "B.Cu") (free) (net 1))
   (via (at 163.195 86.995) (size 0.7) (drill 0.35) (layers "F.Cu" "B.Cu") (free) (net 1))
@@
   (via (at 147.955 86.995) (size 0.7) (drill 0.35) (layers "F.Cu" "B.Cu") (free) (net 1))
   (via (at 152.4 80.645) (size 0.7) (drill 0.35) (layers "F.Cu" "B.Cu") (free) (net 1))
+  (segment (start 146.05 106.045) (end 143.51 103.505) (width 0.2) (layer "B.Cu") (net 1))
+  (segment (start 184.26811 99.05111) (end 184.26811 93.46311) (width 0.2) (layer "B.Cu") (net 1))
+  (segment (start 156.21 106.174711) (end 156.21 108.585) (width 0.2) (layer "B.Cu") (net 1))
+  (segment (start 146.05 107.820289) (end 146.05 106.045) (width 0.2) (layer "B.Cu") (net 1))
+  (segment (start 184.26811 93.46311) (end 184.1706 93.3656) (width 0.2) (layer "B.Cu") (net 1))
+  (segment (start 154.175289 104.14) (end 156.21 106.174711) (width 0.2) (layer "B.Cu") (net 1))
+  (segment (start 146.814711 108.585) (end 146.05 107.820289) (width 0.2) (layer "B.Cu") (net 1))
+  (segment (start 152.4 104.14) (end 154.175289 104.14) (width 0.2) (layer "B.Cu") (net 1))
+  (segment (start 185.547 100.33) (end 184.26811 99.05111) (width 0.2) (layer "B.Cu") (net 1))
+  (segment (start 147.955 108.585) (end 146.814711 108.585) (width 0.2) (layer "B.Cu") (net 1))
   (segment (start 183.007 95.25) (end 179.8575 95.25) (width 0.2) (layer "F.Cu") (net 2))
   (segment (start 185.547 97.79) (end 184.277 96.52) (width 0.2) (layer "F.Cu") (net 3))
@@
   (segment (start 161.29 107.896176) (end 165.1 111.706176) (width 0.2) (layer "F.Cu") (net 43))
   (segment (start 159.125579 104.14) (end 161.29 106.304421) (width 0.2) (layer "F.Cu") (net 43))
-  (segment (start 139.7 101.6) (end 141.8541 103.7541) (width 0.2) (layer "F.Cu") (net 44))
-  (segment (start 141.8541 103.7541) (end 145.9154 103.7541) (width 0.2) (layer "F.Cu") (net 44))
+  (segment (start 139.7 101.6) (end 142.703599 104.603599) (width 0.2) (layer "F.Cu") (net 44))
+  (segment (start 142.703599 104.603599) (end 145.065901 104.603599) (width 0.2) (layer "F.Cu") (net 44))
   (segment (start 167.64 116.8545) (end 168.137 116.8545) (width 0.2) (layer "F.Cu") (net 44))
   (segment (start 168.137 116.8545) (end 168.91 117.6275) (width 0.2) (layer "F.Cu") (net 44))
+  (segment (start 145.065901 104.603599) (end 145.9154 103.7541) (width 0.2) (layer "F.Cu") (net 44))
   (via (at 167.64 116.8545) (size 0.7) (drill 0.35) (layers "F.Cu" "B.Cu") (net 44))
   (segment (start 148.59 105.85721) (end 146.48689 103.7541) (width 0.2) (layer "B.Cu") (net 44))
